File: ESP_WeatherStation.sch (KiCad schematic (older format))
At the start: 19 parts, among them J1 Con1, U1 AZ1117-3.3, U2 ESP-12F, U3 Si7021, U4 BMP280, U5 DS1821C

Commit message: Final version
Parts:
- renumbered R3 to R2, R4 to R3, R5 to R4, R6 to R5, R2 to R6
Connections:
- net +5V: now also J1.8 (Pin_8); no longer J1.7 (Pin_7)
- net BOOT: now also J1.4 (Pin_4); no longer J1.3 (Pin_3)
- net GND: now also J1.1 (Pin_1), J1.3 (Pin_3), J1.7 (Pin_7); no longer J1.2 (Pin_2), J1.4 (Pin_4), J1.8 (Pin_8)
- net RESET: now also J1.2 (Pin_2); no longer J1.1 (Pin_1)
Other:
- moved on the sheet: J1
Changed lines of the file:
@@
 $EndComp
 $Comp
-L R R2
+L R R6
 U 1 1 5A92CA65
 P 2950 2700
-F 0 "R2" V 3030 2700 50  0000 C CNN
+F 0 "R6" V 3030 2700 50  0000 C CNN
 F 1 "10k" V 2950 2700 50  0000 C CNN
 F 2 "Resistors_SMD:R_0603" V 2880 2700 50  0001 C CNN
@@
 $EndComp
 $Comp
-L R R5
+L R R4
 U 1 1 5A92CA9F
 P 5500 2700
-F 0 "R5" V 5550 2550 50  0000 C CNN
+F 0 "R4" V 5550 2550 50  0000 C CNN
 F 1 "1k" V 5500 2700 50  0000 C CNN
 F 2 "Resistors_SMD:R_0603" V 5430 2700 50  0001 C CNN
@@
 L Conn_02x04_Odd_Even J1
 U 1 1 5A92E8C5
-P 4100 4300
-F 0 "J1" H 4150 4500 50  0000 C CNN
-F 1 "Con1" H 4150 4000 50  0000 C CNN
-F 2 "Pin_Headers:Pin_Header_Straight_2x04_Pitch2.54mm_SMD" H 4100 4300 50  0001 C CNN
-F 3 "" H 4100 4300 50  0001 C CNN
-	1    4100 4300
+P 4000 4300
+F 0 "J1" H 4050 4500 50  0000 C CNN
+F 1 "Con1" H 4050 4000 50  0000 C CNN
+F 2 "Pin_Headers:Pin_Header_Straight_2x04_Pitch2.54mm_SMD" H 4000 4300 50  0001 C CNN
+F 3 "" H 4000 4300 50  0001 C CNN
+	1    4000 4300
 	1    0    0    -1
 $EndComp
@@
 	1    0    0    -1
 $EndComp
-Text Label 4750 4400 2    60   ~ 0
+Text Label 3450 4400 0    60   ~ 0
+RXD
+Text Label 4600 4400 2    60   ~ 0
 TXD
-Text Label 3600 4400 0    60   ~ 0
-RXD
 $Comp
 L GND #PWR01
 U 1 1 5A9BD2DC
-P 4500 4650
-F 0 "#PWR01" H 4500 4400 50  0001 C CNN
-F 1 "GND" H 4500 4500 50  0000 C CNN
-F 2 "" H 4500 4650 50  0001 C CNN
-F 3 "" H 4500 4650 50  0001 C CNN
-	1    4500 4650
-	1    0    0    -1
-$EndComp
-Text Label 3600 4300 0    60   ~ 0
+P 3700 4650
+F 0 "#PWR01" H 3700 4400 50  0001 C CNN
+F 1 "GND" H 3700 4500 50  0000 C CNN
+F 2 "" H 3700 4650 50  0001 C CNN
+F 3 "" H 3700 4650 50  0001 C CNN
+	1    3700 4650
+	-1   0    0    -1
+$EndComp
+Text Label 4600 4300 2    60   ~ 0
 BOOT
-Text Label 3600 4200 0    60   ~ 0
+Text Label 4600 4200 2    60   ~ 0
 RESET
 $Comp
 L +5V #PWR02
 U 1 1 5A9BD3F2
-P 3450 4500
-F 0 "#PWR02" H 3450 4350 50  0001 C CNN
-F 1 "+5V" H 3450 4640 50  0000 C CNN
-F 2 "" H 3450 4500 50  0001 C CNN
-F 3 "" H 3450 4500 50  0001 C CNN
-	1    3450 4500
-	1    0    0    -1
+P 4750 4500
+F 0 "#PWR02" H 4750 4350 50  0001 C CNN
+F 1 "+5V" H 4750 4640 50  0000 C CNN
+F 2 "" H 4750 4500 50  0001 C CNN
+F 3 "" H 4750 4500 50  0001 C CNN
+	1    4750 4500
+	-1   0    0    -1
 $EndComp
 $Comp
@@
 SCL
 $Comp
-L R R6
+L R R5
 U 1 1 5A9C2339
 P 5550 2800
-F 0 "R6" V 5600 2650 50  0000 C CNN
+F 0 "R5" V 5600 2650 50  0000 C CNN
 F 1 "10k" V 5550 2800 50  0000 C CNN
 F 2 "Resistors_SMD:R_0603" V 5480 2800 50  0001 C CNN
@@
 SDA
 $Comp
-L R R4
+L R R3
 U 1 1 5A9C3417
 P 2000 2850
-F 0 "R4" V 1900 2850 50  0000 C CNN
+F 0 "R3" V 1900 2850 50  0000 C CNN
 F 1 "82" V 2000 2850 50  0000 C CNN
 F 2 "Resistors_SMD:R_0603" V 1930 2850 50  0001 C CNN
@@
 	5100 2900 5500 2900
 Wire Wire Line
-	3900 4200 3600 4200
-Wire Wire Line
-	3600 4300 3900 4300
-Wire Wire Line
-	3600 4400 3900 4400
-Wire Wire Line
-	4400 4200 4500 4200
-Wire Wire Line
-	4500 4200 4500 4650
-Wire Wire Line
-	4400 4300 4500 4300
-Connection ~ 4500 4300
-Wire Wire Line
-	4400 4500 4500 4500
-Connection ~ 4500 4500
-Wire Wire Line
-	4400 4400 4750 4400
-Wire Wire Line
-	3900 4500 3450 4500
+	4300 4200 4600 4200
+Wire Wire Line
+	4600 4300 4300 4300
+Wire Wire Line
+	4600 4400 4300 4400
+Wire Wire Line
+	3800 4200 3700 4200
+Wire Wire Line
+	3700 4200 3700 4650
+Wire Wire Line
+	3800 4300 3700 4300
+Connection ~ 3700 4300
+Wire Wire Line
+	3800 4500 3700 4500
+Connection ~ 3700 4500
+Wire Wire Line
+	3800 4400 3450 4400
+Wire Wire Line
+	4300 4500 4750 4500
 Wire Wire Line
 	1200 1600 1200 1700
@@
 DATA
 $Comp
-L R R3
+L R R2
 U 1 1 5A9C9735
 P 5450 2500
-F 0 "R3" V 5530 2500 50  0000 C CNN
+F 0 "R2" V 5530 2500 50  0000 C CNN
 F 1 "4.7k" V 5450 2500 50  0000 C CNN
 F 2 "Resistors_SMD:R_0603" V 5380 2500 50  0001 C CNN
